File: eagle_/Laser_Teensy_proto_edits_11-21.brd (EAGLE design)
At the start: 115.6 x 109.2 mm, 145 parts, among them IC1 4051D, IC10 TL074D, IC2 LM1117-3.3, IC3 LM4040B10, IC4 TL074D, IC5 CS42448-CQZ, IC6 MCP6002, IC7 CAT811TTBI-GT3, IC8 MCP6002, IC9 4051D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

Commit message: first commit PAT from mac
Parts:
- added J1: (no value), SparkFun-Connectors:2X13
- moved JP2 22.7 mm to (167.0, 58.9)
- moved X1 10.2 mm to (185.2, 33.3)
- moved R16 0.90 mm to (161.9, 41.3)
- moved R21 0.76 mm to (161.9, 44.0)
- moved R20 0.76 mm to (161.9, 38.5)
- moved R24 0.67 mm to (161.9, 46.8)
- moved R19 0.67 mm to (161.9, 35.8)
- moved R35 0.64 mm to (161.9, 49.5)
- moved R18 0.63 mm to (161.9, 33.0)
- renumbered Y_AUDIO1 to Y_AUDIO
Connections:
- new net N$12: J1.1
- new net N$53: J1.3
- new net N$54: J1.5
- new net N$55: J1.7
- new net N$56: J1.9
- new net N$57: J1.11
- new net N$58: J1.13
- new net N$59: J1.25
- new net N$60: J1.26
- new net N$64: J1.2
Other:
- outline, holes or cut-outs redrawn
